File: order66-lp/pcb/order66-lp.kicad_sch (KiCad schematic)
At the start: 275 parts, among them J1 Battery JST PH, J2 SWD horizontal, J3 SWD millmax vertical, Q1 AO3401A, Q2 BSS138, SW1 CHOC_V1_HS, SW10 CHOC_V1_HS, SW11 CHOC_V1_HS, SW12 CHOC_V1_HS, SW13 CHOC_V1_HS, SW14 CHOC_V1_HS, SW15 CHOC_V1_HS, SW16 CHOC_V1_HS, SW17 CHOC_V1_HS, SW18 CHOC_V1_HS, SW19 CHOC_V1_HS, SW2 CHOC_V1_HS, SW20 CHOC_V1_HS, SW21 CHOC_V1_HS, SW22 CHOC_V1_HS, SW23 CHOC_V1_HS, SW24 CHOC_V1_HS, SW25 CHOC_V1_HS, SW26 CHOC_V1_HS, SW27 CHOC_V1_HS, SW28 CHOC_V1_HS, SW29 CHOC_V1_HS, SW3 CHOC_V1_HS, SW30 CHOC_V1_HS, SW31 CHOC_V1_HS, SW32 CHOC_V1_HS, SW33 CHOC_V1_HS, SW34 CHOC_V1_HS, SW35 CHOC_V1_HS, SW36 CHOC_V1_HS, SW37 CHOC_V1_HS, SW38 CHOC_V1_HS, SW39 CHOC_V1_HS, SW4 CHOC_V1_HS, SW40 CHOC_V1_HS, SW41 CHOC_V1_HS, SW42 CHOC_V1_HS, SW43 CHOC_V1_HS, SW44 CHOC_V1_HS, SW45 CHOC_V1_HS, SW46 CHOC_V1_HS, SW47 CHOC_V1_HS, SW48 CHOC_V1_HS, SW49 CHOC_V1_HS, SW5 CHOC_V1_HS, SW50 CHOC_V1_HS, SW51 CHOC_V1_HS, SW52 CHOC_V1_HS, SW53 CHOC_V1_HS, SW54 CHOC_V1_HS, SW55 CHOC_V1_HS, SW56 CHOC_V1_HS, SW57 CHOC_V1_HS, SW58 CHOC_V1_HS, SW59 CHOC_V1_HS, SW6 CHOC_V1_HS, SW60 CHOC_V1_HS, SW61 RESET, SW62 EG1206A, SW63 SSSS811101, SW7 CHOC_V1_HS, SW8 CHOC_V1_HS, SW9 CHOC_V1_HS, U1 nice!nano v2, U2 TPS61085DGK, U3 74AHCT1G125

Commit message: order66-lp: PCB layout, footprint library, and generator scripts
Adds the previously-untracked half of the low-profile redesign: the
order66-lp.kicad_pcb layout itself, the order66lp.pretty footprint library
(nice!nano header), and the gen_pcb / gen_overlay / gen_nano_footprint /
check_pcb tools, alongside updates to the schematic, BOM, ZMK shield and
existing generators.

Co-Authored-By: Claude Opus 5 (1M context) <noreply@anthropic.com>
Parts:
- added D62: 1N4148WS, Diode_SMD:D_SOD-323, symbol Diode:1N4148WS
- added D63: MBRA340, Diode_SMD:D_SMA, symbol Diode:MBRA340
- added J4: Cirque FFC, marbastlib-various:CON_FH33J-12S-0.5SH, symbol Connector_Generic:Conn_01x12
- added R10, R9: 4k7, Resistor_SMD:R_0402_1005Metric, symbol Device:R
- added SW64: EG1206A, EG1206A:EG1206A_EWI, symbol EG1206A:EG1206A
- added SW65: SSSS811101, SSSS811101:SW_SSSS811101, symbol SSSS811101:SSSS811101
- D61: value MBRA340 -> 1N4148WS; footprint Diode_SMD:D_SMA -> Diode_SMD:D_SOD-323; symbol Diode:MBRA340 -> Diode:1N4148WS
- SW61: value RESET -> MOUSE_BTN; footprint Button_Switch_THT:SW_TH_Tactile_Omron_B3F-100x -> marbastlib-choc:SW_choc_v1_HS_CPG135001S30_1u; symbol Switch:SW_Push -> marbastlib-choc:choc_v1_SW_HS_CPG135001S30
- SW62: value EG1206A -> MOUSE_BTN; footprint EG1206A:EG1206A_EWI -> marbastlib-choc:SW_choc_v1_HS_CPG135001S30_1u; symbol EG1206A:EG1206A -> marbastlib-choc:choc_v1_SW_HS_CPG135001S30
- SW63: value SSSS811101 -> RESET; footprint SSSS811101:SW_SSSS811101 -> Button_Switch_THT:SW_TH_Tactile_Omron_B3F-100x; symbol SSSS811101:SSSS811101 -> Switch:SW_Push
- U1: footprint nice-nano-kicad:nice_nano -> order66lp:nice_nano_Hdr_TH1-12_SMD13-33
Connections:
- net BATT+: now also SW64.2, SW65.1; no longer SW62.2, SW63.1
- net BST_SW: now also D63.2 (A); no longer D61.2 (A)
- net COL0: now also SW19.2, SW31.2, SW43.2, SW55.2, SW61.2, SW7.2
- net COL1: now also SW20.2, SW32.2, SW44.2, SW56.2, SW62.2, SW8.2
- net COL2: now also SW21.2, SW33.2, SW45.2, SW57.2, SW9.2
- net COL3: now also SW10.2, SW22.2, SW34.2, SW46.2, SW58.2
- net COL4: now also SW11.2, SW23.2, SW35.2, SW47.2, SW59.2
- net COL5: now also SW12.2, SW24.2, SW36.2, SW48.2, SW60.2
- net GND: now also SW63.2, J4.11 (Pin_11); no longer SW61.2
- net ROW0: no longer D10.1 (K), D11.1 (K), D12.1 (K), D7.1 (K), D8.1 (K), D9.1 (K)
- net ROW1: no longer D19.1 (K), D20.1 (K), D21.1 (K), D22.1 (K), D23.1 (K), D24.1 (K)
- net ROW2: no longer D31.1 (K), D32.1 (K), D33.1 (K), D34.1 (K), D35.1 (K), D36.1 (K)
- net ROW3: no longer D43.1 (K), D44.1 (K), D45.1 (K), D46.1 (K), D47.1 (K), D48.1 (K)
- net ROW4: no longer D55.1 (K), D56.1 (K), D57.1 (K), D58.1 (K), D59.1 (K), D60.1 (K)
- net RST: now also SW63.1; no longer SW61.1
- net VBATT+: now also SW64.3, SW65.2; no longer SW62.3, SW63.2
- net VCC: now also J4.12 (Pin_12), R10.1, R9.1
- net VLED: now also D63.1 (K); no longer D61.1 (K)
- net TP_DR: now reaches U1.18 (AIN0/P0.02)
- net TP_DR: now also J4.4 (Pin_4)
- net TP_SDA: now reaches U1.5 (P0.17)
- net TP_SDA: now also J4.10 (Pin_10), R9.2
- net TP_SCL: now reaches U1.6 (P0.20)
- net TP_SCL: now also J4.9 (Pin_9), R10.2
- net at SW62.1: now also D62.2 (A)
- removed net COL10: SW11.2, SW23.2, SW35.2, SW47.2, SW59.2, U1.12 (P1.06)
- removed net COL11: SW12.2, SW24.2, SW36.2, SW48.2, SW60.2, U1.31 (P1.01)
- removed net COL6: SW19.2, SW31.2, SW43.2, SW55.2, SW7.2, U1.10 (P0.11)
- removed net COL7: SW20.2, SW32.2, SW44.2, SW56.2, SW8.2, U1.32 (P1.02)
- removed net COL8: SW21.2, SW33.2, SW45.2, SW57.2, SW9.2, U1.33 (P1.07)
- removed net COL9: SW10.2, SW22.2, SW34.2, SW46.2, SW58.2, U1.11 (P1.04)
- new net: D61.2 (A), SW61.1
- new net ROW10: D61.1 (K), D62.1 (K), U1.31 (P1.01)
- new net ROW5: D10.1 (K), D11.1 (K), D12.1 (K), D7.1 (K), D8.1 (K), D9.1 (K), U1.10 (P0.11)
- new net ROW6: D19.1 (K), D20.1 (K), D21.1 (K), D22.1 (K), D23.1 (K), D24.1 (K), U1.32 (P1.02)
- new net ROW7: D31.1 (K), D32.1 (K), D33.1 (K), D34.1 (K), D35.1 (K), D36.1 (K), U1.33 (P1.07)
- new net ROW8: D43.1 (K), D44.1 (K), D45.1 (K), D46.1 (K), D47.1 (K), D48.1 (K), U1.11 (P1.04)
- new net ROW9: D55.1 (K), D56.1 (K), D57.1 (K), D58.1 (K), D59.1 (K), D60.1 (K), U1.12 (P1.06)
- no-connect marks 6 -> 10
Other:
- note added: "KEY MATRIX -- 5 x 12 physical keys on a 11 row x 6 col matrix, col2row. Left half -> rows 0-4, right half -> rows 5-9, mouse buttons -> row 10."
- note added: "MOUSE BUTTONS -- electrical row 10; cols 2-5 of that row are spare"
- note added: "TRACKPAD -- Cirque TM040040, I2C @ 0x2a. Remove the module's R1 to select I2C. Pins 1/2/3/5 are SPI-only; 6/7/8 are its hardware buttons."
- note removed: "KEY MATRIX -- 5 rows x 12 cols, 60 keys, col2row (COL -> switch -> diode anode, cathode -> ROW)"
- moved on the sheet: D61, SW61
